File: ESPRelay.kicad_pcb (KiCad board)
At the start: 2 copper layers, 49 x 81 mm, 25 parts, among them J1 RELAY1, J2 RELAY2, J3 SENSOR_1, J4 SENSOR_2, K1 G5Q-1, K2 G5Q-1, Q1 2N3904, Q2 2N3904, U1 NodeMCU_1.0_(ESP-12E), U2 EL817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

Commit message: Removed offensive message on silkscreen
Other:
- board text removed: "Fuck Trump"
